File: trackball.kicad_sch (KiCad schematic)
At the start: 174 parts, among them J1 ZX-PM2.0-2-4PY, SW1 HX TC-5608-Y, SW2 HX TC-5608-Y, SW3 HX TC-5608-Y, SW4 HX TC-5608-Y, SW5 HX TC-5608-Y, SW6 HX TC-5608-Y, SW7 HX TC-5608-Y, SW8 HX TC-5608-Y, U1 SY8089A1AAC, U10 WS2812B, U11 WS2812B, U12 WS2812B, U13 WS2812B, U14 WS2812B, U15 WS2812B, U16 WS2812B, U17 WS2812B, U18 WS2812B, U19 WS2812B, U2 USB-TYPE-C-017, U20 WS2812B, U3 PMW3610, U4 PMW3610, U5 WS2812B, U6 WS2812B, U7 WS2812B, U8 WS2812B, U9 WS2812B, X1 XL7EL89CKI-111YLC-32M

Commit message: chore: checkpoint
Parts:
- AE1: footprint antenna:Texas_SWRA117D_2.4GHz_Right -> antenna:Texas_SWRA117D_2.4GHz_Left
Connections:
- net CHG_IRQ: now also U_MCU1.A16 (P1.05); no longer U_MCU1.N1 (P0.08)
- net CHG_ISACTIVE: now also U_MCU1.B15 (P1.03); no longer U_MCU1.L1 (P0.06)
- net CHG_SCL: now also U_MCU1.B17 (P0.23); no longer U_MCU1.L24 (P0.09/NFC1)
- net CHG_SDA: now also U_MCU1.A20 (P0.25); no longer U_MCU1.M2 (P0.07/TRACECLK)
- net MCU_LED1: now also U_MCU1.L24 (P0.09/NFC1); no longer U_MCU1.P2 (P1.08)
- net MCU_LED2: now also U_MCU1.Y23 (P1.01); no longer U_MCU1.R1 (P1.09/TRACEDATA3)
- net MCU_LED3: now also U_MCU1.AD20 (P0.24); no longer U_MCU1.W24 (P1.02)
- net MCU_SWO: now also J1.3
- net RE1_A: now also U_MCU1.AD12 (P0.17); no longer U_MCU1.U24 (P1.04)
- net RE1_B: now also U_MCU1.AC11 (P0.16); no longer U_MCU1.U1 (P0.12/TRACEDATA1)
- net RE1_SW: now also U_MCU1.AD10 (P0.15); no longer U_MCU1.AC9 (P0.14)
- net RE2_A: now also U_MCU1.P2 (P1.08); no longer U_MCU1.T2 (P0.11/TRACEDATA2)
- net RE2_B: now also U_MCU1.R1 (P1.09/TRACEDATA3); no longer U_MCU1.R24 (P1.6)
- net RE2_SW: now also U_MCU1.T2 (P0.11/TRACEDATA2); no longer U_MCU1.Y23 (P1.01)
- net RGB_DOUT: now also U_MCU1.U1 (P0.12/TRACEDATA1); no longer U_MCU1.A20 (P0.25)
- net SS1_CLK: now also U_MCU1.B11 (P0.28/AIN4); no longer U_MCU1.A14 (P0.19)
- net SS1_DIO: now also U_MCU1.B13 (P0.03/AIN1); no longer U_MCU1.A12 (P0.02/AIN0)
- net SS1_MTN: now also U_MCU1.A12 (P0.02/AIN0); no longer U_MCU1.F2 (P0.01/XL2)
- net SS1_NCS: now also U_MCU1.B9 (P0.30/AIN6); no longer U_MCU1.A16 (P1.05)
- net SS1_RST: no longer J1.3
- net SS2_CLK: now also U_MCU1.L1 (P0.06); no longer U_MCU1.H2 (P0.27)
- net SS2_DIO: now also U_MCU1.J24 (P0.10/NFC2); no longer U_MCU1.G1 (P0.26)
- net SS2_MTN: now also U_MCU1.U24 (P1.04); no longer U_MCU1.K2 (P0.05/AIN3)
- net SS2_NCS: now also U_MCU1.P23 (P1.07); no longer U_MCU1.J1 (P0.04/AIN2)
- net SS2_RST: now also U_MCU1.R24 (P1.6); no longer J1.8, U_MCU1.J24 (P0.10/NFC2)
- net SW1: now also U_MCU1.G1 (P0.26); no longer U_MCU1.AD20 (P0.24)
- net SW2: now also U_MCU1.H2 (P0.27); no longer U_MCU1.AD18 (P0.22)
- net SW3: now also U_MCU1.F2 (P0.01/XL2); no longer U_MCU1.AD16 (P0.20)
- net SW4: now also U_MCU1.AC17 (P0.21); no longer U_MCU1.AD12 (P0.17)
- net SW5: now also U_MCU1.N1 (P0.08); no longer U_MCU1.AD10 (P0.15)
- net SW6: now also U_MCU1.M2 (P0.07/TRACECLK); no longer U_MCU1.AD8 (P0.13)
- net SW7: now also U_MCU1.K2 (P0.05/AIN3); no longer U_MCU1.AC17 (P0.21)
- net SW8: now also U_MCU1.J1 (P0.04/AIN2); no longer U_MCU1.AC11 (P0.16)
- net USB_MUX_SEL: now also U_MCU1.A14 (P0.19); no longer U_MCU1.P23 (P1.07)
- no-connect marks 52 -> 53
Other:
- moved on the sheet: C23, C26, C27

Commit message: chore: checkpoint
Connections:
- net RE1_A: no longer C19.1, FPC6.3, R21.2, U_RE1.A
- net RE1_B: no longer C20.2, FPC6.5, R24.1, U_RE1.B
- net RE1_SW: no longer C13.2, FPC6.2, R19.2
- net RE2_A: no longer C37.1, FPC8.3, R37.2, U_RE2.A
- net RE2_B: no longer C38.2, FPC8.5, R38.1, U_RE2.B
- net RE2_SW: no longer C28.2, FPC8.2, R31.2
- net SS1_CLK: no longer FPC2.3, U3.3 (SCLK)
- net SS1_DIO: no longer FPC2.2, U3.2 (SDIO)
- net SS1_MTN: no longer FPC2.6, U3.8 (MOTION)
- net SS1_NCS: no longer FPC2.4, U3.5 (NCS)
- net SS1_RST: no longer FPC2.5, R45.1, U3.7 (NRESET)
- net SS2_CLK: no longer FPC4.3, U4.3 (SCLK)
- net SS2_DIO: no longer FPC4.2, U4.2 (SDIO)
- net SS2_MTN: no longer FPC4.6, U4.8 (MOTION)
- net SS2_NCS: no longer FPC4.4, U4.5 (NCS)
- net SS2_RST: no longer FPC4.5, R48.1, U4.7 (NRESET)
- new net D_RE1_A: C19.1, FPC6.3, R21.2, U_RE1.A
- new net D_RE1_B: C20.2, FPC6.5, R24.1, U_RE1.B
- new net D_RE1_SW: C13.2, FPC6.2, R19.2
- new net D_RE2_A: C37.1, FPC8.3, R37.2, U_RE2.A
- new net D_RE2_B: C38.2, FPC8.5, R38.1, U_RE2.B
- new net D_RE2_SW: C28.2, FPC8.2, R31.2
- new net D_SS1_CLK: FPC2.3, U3.3 (SCLK)
- new net D_SS1_DIO: FPC2.2, U3.2 (SDIO)
- new net D_SS1_MTN: FPC2.6, U3.8 (MOTION)
- new net D_SS1_NCS: FPC2.4, U3.5 (NCS)
- new net D_SS1_RST: FPC2.5, R45.1, U3.7 (NRESET)
- new net D_SS2_CLK: FPC4.3, U4.3 (SCLK)
- new net D_SS2_DIO: FPC4.2, U4.2 (SDIO)
- new net D_SS2_MTN: FPC4.6, U4.8 (MOTION)
- new net D_SS2_NCS: FPC4.4, U4.5 (NCS)
- new net D_SS2_RST: FPC4.5, R48.1, U4.7 (NRESET)
Changed lines of the file:
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@@
 		)
 	)
-	(global_label "SS1_MTN"
+	(global_label "D_SS1_MTN"
 		(shape bidirectional)
 		(at 83.82 55.88 180)
@@
 		)
 		(property "Intersheetrefs" "${INTERSHEET_REFS}"
-			(at 71.3779 55.88 0)
+			(at 69.1403 55.88 0)
 			(effects
 				(font
@@
 		)
 	)
-	(global_label "SS1_RST"
+	(global_label "D_SS1_RST"
 		(shape bidirectional)
 		(at 83.82 53.34 180)
@@
 		)
 		(property "Intersheetrefs" "${INTERSHEET_REFS}"
-			(at 71.6803 53.34 0)
+			(at 69.4427 53.34 0)
 			(effects
 				(font
@@
 		)
 	)
-	(global_label "SS2_NCS"
+	(global_label "D_SS2_NCS"
 		(shape bidirectional)
 		(at 83.82 95.25 180)
@@
 		)
 		(property "Intersheetrefs" "${INTERSHEET_REFS}"
-			(at 71.3174 95.25 0)
+			(at 69.0798 95.25 0)
 			(effects
 				(font
@@
 		)
 	)
-	(global_label "RE2_SW"
+	(global_label "D_RE2_SW"
 		(shape bidirectional)
 		(at 83.82 179.07 180)
@@
 		)
 		(property "Intersheetrefs" "${INTERSHEET_REFS}"
-			(at 72.4665 179.07 0)
+			(at 70.2289 179.07 0)
 			(effects
 				(font
@@
 		)
 	)
-	(global_label "SS1_CLK"
+	(global_label "D_SS1_CLK"
 		(shape bidirectional)
 		(at 83.82 48.26 180)
@@
 		)
 		(property "Intersheetrefs" "${INTERSHEET_REFS}"
-			(at 71.5593 48.26 0)
+			(at 69.3217 48.26 0)
 			(effects
 				(font
@@
 		)
 	)
-	(global_label "RE1_SW"
+	(global_label "D_RE1_SW"
 		(shape bidirectional)
 		(at 480.06 125.73 0)
@@
 		)
 		(property "Intersheetrefs" "${INTERSHEET_REFS}"
-			(at 491.4135 125.73 0)
+			(at 493.6511 125.73 0)
 			(effects
 				(font
@@
 		)
 	)
-	(global_label "SS1_DIO"
+	(global_label "D_SS1_DIO"
 		(shape bidirectional)
 		(at 83.82 45.72 180)
@@
 		)
 		(property "Intersheetrefs" "${INTERSHEET_REFS}"
-			(at 71.9221 45.72 0)
+			(at 69.6845 45.72 0)
 			(effects
 				(font
@@
 		)
 	)
-	(global_label "SS2_MTN"
+	(global_label "D_SS2_MTN"
 		(shape bidirectional)
 		(at 431.8 359.41 180)
@@
 		)
 		(property "Intersheetrefs" "${INTERSHEET_REFS}"
-			(at 419.3579 359.41 0)
+			(at 417.1203 359.41 0)
 			(effects
 				(font
@@
 		)
 	)
-	(global_label "SS2_CLK"
+	(global_label "D_SS2_CLK"
 		(shape bidirectional)
 		(at 83.82 92.71 180)
@@
 		)
 		(property "Intersheetrefs" "${INTERSHEET_REFS}"
-			(at 71.5593 92.71 0)
+			(at 69.3217 92.71 0)
 			(effects
 				(font
@@
 		)
 	)
-	(global_label "RE1_A"
+	(global_label "D_RE1_A"
 		(shape bidirectional)
 		(at 83.82 137.16 180)
@@
 		)
 		(property "Intersheetrefs" "${INTERSHEET_REFS}"
-			(at 74.0388 137.16 0)
+			(at 71.8012 137.16 0)
 			(effects
 				(font
@@
 		)
 	)
-	(global_label "SS2_RST"
+	(global_label "D_SS2_RST"
 		(shape bidirectional)
 		(at 431.8 356.87 180)
@@
 		)
 		(property "Intersheetrefs" "${INTERSHEET_REFS}"
-			(at 419.6603 356.87 0)
+			(at 417.4227 356.87 0)
 			(effects
 				(font
@@
 		)
 	)
-	(global_label "RE2_SW"
+	(global_label "D_RE2_SW"
 		(shape bidirectional)
 		(at 480.06 193.04 0)
@@
 		)
 		(property "Intersheetrefs" "${INTERSHEET_REFS}"
-			(at 491.4135 193.04 0)
+			(at 493.6511 193.04 0)
 			(effects
 				(font
@@
 		)
 	)
-	(global_label "SS2_NCS"
+	(global_label "D_SS2_NCS"
 		(shape bidirectional)
 		(at 431.8 351.79 180)
@@
 		)
 		(property "Intersheetrefs" "${INTERSHEET_REFS}"
-			(at 419.2974 351.79 0)
+			(at 417.0598 351.79 0)
 			(effects
 				(font
@@
 		)
 	)
-	(global_label "SS2_DIO"
+	(global_label "D_SS2_DIO"
 		(shape bidirectional)
 		(at 83.82 90.17 180)
@@
 		)
 		(property "Intersheetrefs" "${INTERSHEET_REFS}"
-			(at 71.9221 90.17 0)
+			(at 69.6845 90.17 0)
 			(effects
 				(font
@@
 		)
 	)
-	(global_label "RE1_SW"
+	(global_label "D_RE1_SW"
 		(shape bidirectional)
 		(at 83.82 134.62 180)
@@
 		)
 		(property "Intersheetrefs" "${INTERSHEET_REFS}"
-			(at 72.4665 134.62 0)
+			(at 70.2289 134.62 0)
 			(effects
 				(font
@@
 		)
 	)
-	(global_label "SS2_RST"
+	(global_label "D_SS2_RST"
 		(shape bidirectional)
 		(at 481.33 402.59 180)
@@
 		)
 		(property "Intersheetrefs" "${INTERSHEET_REFS}"
-			(at 469.1903 402.59 0)
+			(at 466.9527 402.59 0)
 			(effects
 				(font
@@
 		)
 	)
-	(global_label "SS1_DIO"
+	(global_label "D_SS1_DIO"
 		(shape bidirectional)
 		(at 431.8 290.83 180)
@@
 		)
 		(property "Intersheetrefs" "${INTERSHEET_REFS}"
-			(at 419.9021 290.83 0)
+			(at 417.6645 290.83 0)
 			(effects
 				(font
@@
 		)
 	)
-	(global_label "SS1_RST"
+	(global_label "D_SS1_RST"
 		(shape bidirectional)
 		(at 481.33 393.7 180)
@@
 		)
 		(property "Intersheetrefs" "${INTERSHEET_REFS}"
-			(at 469.1903 393.7 0)
+			(at 466.9527 393.7 0)
 			(effects
 				(font
@@
 		)
 	)
-	(global_label "RE2_B"
+	(global_label "D_RE2_B"
 		(shape bidirectional)
 		(at 83.82 186.69 180)
@@
 		)
 		(property "Intersheetrefs" "${INTERSHEET_REFS}"
-			(at 73.8574 186.69 0)
+			(at 71.6198 186.69 0)
 			(effects
 				(font
@@
 		)
 	)
-	(global_label "SS2_RST"
+	(global_label "D_SS2_RST"
 		(shape bidirectional)
 		(at 83.82 97.79 180)
@@
 		)
 		(property "Intersheetrefs" "${INTERSHEET_REFS}"
-			(at 71.6803 97.79 0)
+			(at 69.4427 97.79 0)
 			(effects
 				(font
@@
 		)
 	)
-	(global_label "RE2_A"
+	(global_label "D_RE2_A"
 		(shape bidirectional)
 		(at 83.82 181.61 180)
@@
 		)
 		(property "Intersheetrefs" "${INTERSHEET_REFS}"
-			(at 74.0388 181.61 0)
+			(at 71.8012 181.61 0)
 			(effects
 				(font
@@
 		)
 	)
-	(global_label "RE2_A"
+	(global_label "D_RE2_A"
 		(shape bidirectional)
 		(at 462.28 227.33 180)
@@
 		)
 		(property "Intersheetrefs" "${INTERSHEET_REFS}"
-			(at 452.4988 227.33 0)
+			(at 450.2612 227.33 0)
 			(effects
 				(font
@@
 		)
 	)
-	(global_label "SS1_NCS"
+	(global_label "D_SS1_NCS"
 		(shape bidirectional)
 		(at 83.82 50.8 180)
@@
 		)
 		(property "Intersheetrefs" "${INTERSHEET_REFS}"
-			(at 71.3174 50.8 0)
+			(at 69.0798 50.8 0)
 			(effects
 				(font
@@
 		)
 	)
-	(global_label "SS1_MTN"
+	(global_label "D_SS1_MTN"
 		(shape bidirectional)
 		(at 431.8 306.07 180)
@@
 		)
 		(property "Intersheetrefs" "${INTERSHEET_REFS}"
-			(at 419.3579 306.07 0)
+			(at 417.1203 306.07 0)
 			(effects
 				(font
@@
 		)
 	)
-	(global_label "RE1_B"
+	(global_label "D_RE1_B"
 		(shape bidirectional)
 		(at 83.82 142.24 180)
@@
 		)
 		(property "Intersheetrefs" "${INTERSHEET_REFS}"
-			(at 73.8574 142.24 0)
+			(at 71.6198 142.24 0)
 			(effects
 				(font
@@
 		)
 	)
-	(global_label "RE1_B"
+	(global_label "D_RE1_B"
 		(shape bidirectional)
 		(at 486.41 163.83 0)
@@
 		)
 		(property "Intersheetrefs" "${INTERSHEET_REFS}"
-			(at 496.3726 163.83 0)
+			(at 498.6102 163.83 0)
 			(effects
 				(font
@@
 		)
 	)
-	(global_label "SS2_MTN"
+	(global_label "D_SS2_MTN"
 		(shape bidirectional)
 		(at 83.82 100.33 180)
@@
 		)
 		(property "Intersheetrefs" "${INTERSHEET_REFS}"
-			(at 71.3779 100.33 0)
+			(at 69.1403 100.33 0)
 			(effects
 				(font
@@
 		)
 	)
-	(global_label "RE2_B"
+	(global_label "D_RE2_B"
 		(shape bidirectional)
 		(at 486.41 231.14 0)
@@
 		)
 		(property "Intersheetrefs" "${INTERSHEET_REFS}"
-			(at 496.3726 231.14 0)
+			(at 498.6102 231.14 0)
 			(effects
 				(font
@@
 		)
 	)
-	(global_label "SS2_CLK"
+	(global_label "D_SS2_CLK"
 		(shape bidirectional)
 		(at 431.8 346.71 180)
@@
 		)
 		(property "Intersheetrefs" "${INTERSHEET_REFS}"
-			(at 419.5393 346.71 0)
+			(at 417.3017 346.71 0)
 			(effects
 				(font
@@
 		)
 	)
-	(global_label "SS1_NCS"
+	(global_label "D_SS1_NCS"
 		(shape bidirectional)
 		(at 431.8 298.45 180)
@@
 		)
 		(property "Intersheetrefs" "${INTERSHEET_REFS}"
-			(at 419.2974 298.45 0)
+			(at 417.0598 298.45 0)
 			(effects
 				(font
@@
 		)
 	)
-	(global_label "SS2_DIO"
+	(global_label "D_SS2_DIO"
 		(shape bidirectional)
 		(at 431.8 344.17 180)
@@
 		)
 		(property "Intersheetrefs" "${INTERSHEET_REFS}"
-			(at 419.9021 344.17 0)
+			(at 417.6645 344.17 0)
 			(effects
 				(font
@@
 		)
 	)
-	(global_label "SS1_RST"
+	(global_label "D_SS1_RST"
 		(shape bidirectional)
 		(at 431.8 303.53 180)
@@
 		)
 		(property "Intersheetrefs" "${INTERSHEET_REFS}"
-			(at 419.6603 303.53 0)
+			(at 417.4227 303.53 0)
 			(effects
 				(font
@@
 		)
 	)
-	(global_label "SS1_CLK"
+	(global_label "D_SS1_CLK"
 		(shape bidirectional)
 		(at 431.8 293.37 180)
@@
 		)
 		(property "Intersheetrefs" "${INTERSHEET_REFS}"
-			(at 419.5393 293.37 0)
+			(at 417.3017 293.37 0)
 			(effects
 				(font
@@
 		)
 	)
-	(global_label "RE1_A"
+	(global_label "D_RE1_A"
 		(shape bidirectional)
 		(at 462.28 160.02 180)
@@
 		)
 		(property "Intersheetrefs" "${INTERSHEET_REFS}"
-			(at 452.4988 160.02 0)
+			(at 450.2612 160.02 0)
 			(effects
 				(font

Commit message: chore: checkpoint
Connections:
- net 1V8: no longer C45.1, C52.1, C60.1, C61.1, FPC2.1, FPC4.1, FPC6.1, FPC8.1, R20.2, R21.1, R24.2, R32.2, R37.1, R38.2, R45.2, R48.2, U3.14 (VDD), U3.6 (VDDIO), U4.14 (VDD), U4.6 (VDDIO)
- net GND: no longer C13.1, C19.2, C20.1, C28.1, C37.2, C38.1, C45.2, C47.1, C48.2, C49.2, C52.2, C53.1, C54.2, C55.2, C60.2, C61.2, FPC2.7, FPC2.8, FPC4.7, FPC4.8, FPC6.7, FPC6.8, FPC8.7, FPC8.8, U3.11 (GND), U4.11 (GND), U_RE1.COM, U_RE1.D, U_RE2.COM, U_RE2.D
- new net D_RE1_1V8: FPC6.1, R20.2, R21.1, R24.2
- new net D_RE1_GND: C13.1, C19.2, C20.1, FPC6.7, FPC6.8, U_RE1.COM, U_RE1.D
- new net D_RE2_1V8: FPC8.1, R32.2, R37.1, R38.2
- new net D_RE2_GND: C28.1, C37.2, C38.1, FPC8.7, FPC8.8, U_RE2.COM, U_RE2.D
- new net D_SS1_1V8: C45.1, C60.1, FPC2.1, R45.2, U3.14 (VDD), U3.6 (VDDIO)
- new net D_SS1_GND: C45.2, C47.1, C48.2, C49.2, C60.2, FPC2.7, FPC2.8, U3.11 (GND)
- new net D_SS2_1V8: C52.1, C61.1, FPC4.1, R48.2, U4.14 (VDD), U4.6 (VDDIO)
- new net D_SS2_GND: C52.2, C53.1, C54.2, C55.2, C61.2, FPC4.7, FPC4.8, U4.11 (GND)
Other:
- moved on the sheet: C13, C14, C15, C17, C18, C19, C20, C24, C25, C28, C32, C33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

Commit message: chore: checkpoint
Parts:
- R1, R10, R15, R16, R20, R21, R22, R23, R24, R27, R28, R3, R32, R33, R34, R37, R38, R39, R4, R40, R41, R42, R45, R48, R54, R55, R9: LCSC Part C364845 -> C273334
Changed lines of the file:
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@@
 			)
 		)
-		(property "LCSC Part" "C364845"
+		(property "LCSC Part" "C273334"
 			(at 207.01 308.61 0)
 			(effects
@@
 			)
 		)
-		(property "LCSC Part" "C364845"
+		(property "LCSC Part" "C273334"
 			(at 464.82 67.31 0)
 			(effects
@@
 			)
 		)
-		(property "LCSC Part" "C364845"
+		(property "LCSC Part" "C273334"
 			(at 288.29 83.82 0)
 			(effects
@@
 			)
 		)
-		(property "LCSC Part" "C364845"
+		(property "LCSC Part" "C273334"
 			(at 424.18 143.51 0)
 			(effects
@@
 			)
 		)
-		(property "LCSC Part" "C364845"
+		(property "LCSC Part" "C273334"
 			(at 223.52 290.83 0)
 			(effects
@@
 			)
 		)
-		(property "LCSC Part" "C364845"
+		(property "LCSC Part" "C273334"
 			(at 378.46 116.84 0)
 			(effects
@@
 			)
 		)
-		(property "LCSC Part" "C364845"
+		(property "LCSC Part" "C273334"
 			(at 299.72 83.82 0)
 			(effects
@@
 			)
 		)
-		(property "LCSC Part" "C364845"
+		(property "LCSC Part" "C273334"
 			(at 474.98 402.59 0)
 			(effects
@@
 			)
 		)
-		(property "LCSC Part" "C364845"
+		(property "LCSC Part" "C273334"
 			(at 464.82 46.99 0)
 			(effects
@@
 			)
 		)
-		(property "LCSC Part" "C364845"
+		(property "LCSC Part" "C273334"
 			(at 424.18 116.84 0)
 			(effects
@@
 			)
 		)
-		(property "LCSC Part" "C364845"
+		(property "LCSC Part" "C273334"
 			(at 474.98 411.48 0)
 			(effects
@@
 			)
 		)
-		(property "LCSC Part" "C364845"
+		(property "LCSC Part" "C273334"
 			(at 462.28 195.58 0)
 			(effects
@@
 			)
 		)
-		(property "LCSC Part" "C364845"
+		(property "LCSC Part" "C273334"
 			(at 485.14 100.33 0)
 			(effects
@@
 			)
 		)
-		(property "LCSC Part" "C364845"
+		(property "LCSC Part" "C273334"
 			(at 365.76 87.63 0)
 			(effects
@@
 			)
 		)
-		(property "LCSC Part" "C364845"
+		(property "LCSC Part" "C273334"
 			(at 462.28 128.27 0)
 			(effects
@@
 			)
 		)
-		(property "LCSC Part" "C364845"
+		(property "LCSC Part" "C273334"
 			(at 207.01 290.83 0)
 			(effects
@@
 			)
 		)
-		(property "LCSC Part" "C364845"
+		(property "LCSC Part" "C273334"
 			(at 491.49 240.03 0)
 			(effects
@@
 			)
 		)
-		(property "LCSC Part" "C364845"
+		(property "LCSC Part" "C273334"
 			(at 444.5 153.67 0)
 			(effects
@@
 			)
 		)
-		(property "LCSC Part" "C364845"
+		(property "LCSC Part" "C273334"
 			(at 424.18 196.85 0)
 			(effects
@@
 			)
 		)
-		(property "LCSC Part" "C364845"
+		(property "LCSC Part" "C273334"
 			(at 491.49 172.72 0)
 			(effects
@@
 			)
 		)
-		(property "LCSC Part" "C364845"
+		(property "LCSC Part" "C273334"
 			(at 378.46 143.51 0)
 			(effects
@@
 			)
 		)
-		(property "LCSC Part" "C364845"
+		(property "LCSC Part" "C273334"
 			(at 223.52 308.61 0)
 			(effects
@@
 			)
 		)
-		(property "LCSC Part" "C364845"
+		(property "LCSC Part" "C273334"
 			(at 378.46 196.85 0)
 			(effects
@@
 			)
 		)
-		(property "LCSC Part" "C364845"
+		(property "LCSC Part" "C273334"
 			(at 424.18 170.18 0)
 			(effects
@@
 			)
 		)
-		(property "LCSC Part" "C364845"
+		(property "LCSC Part" "C273334"
 			(at 444.5 220.98 0)
 			(effects
@@
 			)
 		)
-		(property "LCSC Part" "C364845"
+		(property "LCSC Part" "C273334"
 			(at 464.82 57.15 0)
 			(effects
@@
 			)
 		)
-		(property "LCSC Part" "C364845"
+		(property "LCSC Part" "C273334"
 			(at 378.46 170.18 0)
 			(effects

Commit message: chore: checkpoint
Parts:
- added LED10, LED11, LED12, LED13, LED14, LED7, LED8, LED9: SZYY0402W, easyeda2kicad:LED0402-RD_WHITE, symbol easyeda2kicad:SZYY0402W
- added Q1: SI2302_C2891732, easyeda2kicad:SOT-23-3_L2.9-W1.3-P1.90-LS2.4-BR, symbol easyeda2kicad:SI2302_C2891732
- added R57: FRC0402F1002TS, easyeda2kicad:R0402, symbol easyeda2kicad:FRC0402F1002TS
- added R58, R59, R60, R61, R62, R63, R64, R71: RT0402BRE0750RL, easyeda2kicad:R0402, symbol easyeda2kicad:RT0402BRE0750RL
Connections:
- net 3V3: now also R58.2, R59.2, R60.2, R61.2, R62.2, R63.2, R64.2, R71.2
- net GND: now also Q1.2 (S)
- net MCU_BCKLT_EN: now reaches U_MCU1.AD16 (P0.20)
- net MCU_BCKLT_EN: now also R57.1
- new net: LED13.2 (A), R63.1
- new net: LED7.2 (A), R71.1
- new net: Q1.1 (G), R57.2
- new net: LED12.2 (A), R62.1
- new net: LED9.2 (A), R59.1
- new net: LED11.2 (A), R61.1
- new net: LED14.2 (A), R64.1
- new net: LED10.2 (A), R60.1
- new net: LED8.2 (A), R58.1
- new net BCKLT_GND: LED10.1 (K), LED11.1 (K), LED12.1 (K), LED13.1 (K), LED14.1 (K), LED7.1 (K), LED8.1 (K), LED9.1 (K), Q1.3 (D)
- no-connect marks 53 -> 52
Other:
- moved on the sheet: BAT1, C16, C21, C40, C41, C42, C46, J1, R39, R40, R41, R42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

Commit message: chore: checkpoint
Parts:
- added LED15: PD15-22C/TR8, easyeda2kicad:SENSOR-SMD_PD15-22C-TR8, symbol easyeda2kicad:PD15-22C_TR8
- added R65, R66: FRC0402F1002TS, easyeda2kicad:R0402, symbol easyeda2kicad:FRC0402F1002TS
- added U21: ANT3216LL00R2400A, easyeda2kicad:ANT-SMD_L3.2-W1.6, symbol easyeda2kicad:ANT3216LL00R2400A
Connections:
- net 3V3: now also LED15.1 (C), LED15.4 (C)
- net CHG_ADC: now also LED15.2 (A), LED15.3 (A), R65.2
- net GND: now also R66.1
- new net: R65.1, R66.2
- no-connect marks 52 -> 54
Other:
- note added: "alternative antenna? 5dBi stated"
- moved on the sheet: BAT1, J1, LED10, LED11, LED12, LED13, LED14, LED7, LED8, LED9, R43, R58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
