File: trackball.kicad_pcb (KiCad board)
At the start: 4 copper layers, 65 x 85 mm, 255 parts, among them J2 ZX-PM2.0-2-4PY, Q1 XR2302, Q2 XR2302, Q4 XR2302, SW1 HX TC-5608-Y, SW2 HX TC-5608-Y, SW3 HX TC-5608-Y, SW4 HX TC-5608-Y, SW5 HX TC-5608-Y, SW6 HX TC-5608-Y, SW7 HX TC-5608-Y, SW8 HX TC-5608-Y, SW9 TS-1010-C-A, U1 USB-TYPE-C-017, U10 WS2812B, U11 WS2812B, U12 WS2812B, U13 WS2812B, U14 WS2812B, U15 WS2812B, U16 WS2812B, U17 WS2812B, U18 WS2812B, U19 WS2812B, U2 SY80004DQD, U20 WS2812B, U21 WS2812B, U3 SY80004DQD, U4 PMW3610, U5 PMW3610, U6 WS2812B, U7 WS2812B, U8 WS2812B, U9 WS2812B, X1 XL7EL89CKI-111YLC-32M

Commit message: chore: refactoring
Parts:
- moved FPC3 0.30 mm to (80.3, 54.1)
- moved ? 0.13 mm to (66.4, 61.5)
- moved ? 0.13 mm to (63.4, 61.5)
- moved ? 0.13 mm to (64.2, 61.5)
- moved ? 0.13 mm to (64.9, 61.5)
- moved ? 0.13 mm to (65.6, 61.5)
Routing:
- net 1V8: track 357.1 -> 321.0 mm
- net D_SS2_1V8: track 42.1 -> 22.9 mm
- net D_SS1_1V8: track 42.1 -> 22.9 mm
- net GND: track 81.7 -> 69.5 mm, vias 143 -> 164
- net CHG_USBD_P: track 22.4 -> 23.8 mm
- net MCU_DEC46: track 14.1 -> 13.2 mm
- net USB_MUX_SEL: track 38.7 -> 38.2 mm
- net SW1: track 20.5 -> 21.0 mm
- net 3V3: track 266.1 -> 265.6 mm
Other:
- board text added: "join if no NTC"

Commit message: chore: refactoring
Routing:
- net 1V8: track 321.0 -> 324.7 mm

Commit message: chore: refactoring
Routing:
- net USB_VBUS: track 140.3 -> 148.6 mm
- net GND: track 69.5 -> 68.3 mm, vias 164 -> 166
